Commit message: remove kinect

File: resource/spot_noarm.urdf (robot description, URDF)
Before this commit: robot Spot, 47 links, 46 joints
Links:
- removed link kinect color
- removed link kinect range
- removed link solid
Joints:
- removed joint base_link_solid_joint
- removed joint solid_kinect color_joint
- removed joint solid_kinect range_joint
